Commit message: feat : four color sensors underneath the mBot2

File: mbot2_description/urdf/mbot2.urdf.xacro (robot description, xacro)
@@ -32,4 +32,10 @@
   <xacro:property name="us_height" value="0.020"/>
   <xacro:property name="us_mass"   value="0.01"/>
+  <!-- Quad RGB color sensor array, underside of the chassis -->
+  <xacro:property name="qrgb_size" value="0.008"/>
+  <xacro:property name="qrgb_height" value="0.004"/>
+  <xacro:property name="qrgb_mass"   value="0.001"/>
+  <xacro:property name="qrgb_x" value="0.0"/>
+  <xacro:property name="qrgb_z" value="${wheel_radius - qrgb_height/2}"/>
   <!-- Colors -->
   <material name="mbot_blue">
@@ -221,4 +227,55 @@
   </gazebo>
   <!-- ============================================================ -->
+  <!-- Quad RGB color sensor array (4x), underside of the chassis    -->
+  <!-- Each unit is modeled as a 1x1 pixel downward-facing camera,   -->
+  <!-- matching the real Quad RGB module's per-channel color read.   -->
+  <!-- ============================================================ -->
+  <xacro:macro name="quad_rgb_unit" params="idx y_off">
+    <link name="quad_rgb_${idx}_link">
+      <visual>
+        <geometry>
+          <box size="${qrgb_size} ${qrgb_size} ${qrgb_height}"/>
+        </geometry>
+        <material name="mbot_black"/>
+      </visual>
+      <inertial>
+        <mass value="${qrgb_mass}"/>
+        <inertia ixx="1e-8" ixy="0" ixz="0" iyy="1e-8" iyz="0" izz="1e-8"/>
+      </inertial>
+    </link>
+    <joint name="quad_rgb_${idx}_joint" type="fixed">
+      <parent link="base_link"/>
+      <child link="quad_rgb_${idx}_link"/>
+      <origin xyz="${qrgb_x} ${y_off} ${qrgb_z}" rpy="0 0 0"/>
+    </joint>
+    <gazebo reference="quad_rgb_${idx}_link">
+      <sensor name="quad_rgb_${idx}_sensor" type="camera">
+        <!-- pitch +90deg: rotates the sensor's forward (+x) axis to point straight down (-z) -->
+        <pose>0 0 0 0 1.5707963 0</pose>
+        <topic>quad_rgb/${idx}/image</topic>
+        <update_rate>15</update_rate>
+        <always_on>true</always_on>
+        <visualize>false</visualize>
+        <camera>
+          <horizontal_fov>0.5</horizontal_fov>
+          <image>
+            <width>1</width>
+            <height>1</height>
+            <format>R8G8B8</format>
+          </image>
+          <clip>
+            <!-- far must be >= 0.1 (Gazebo Fortress camera clip minimum) -->
+            <near>0.01</near>
+            <far>0.15</far>
+          </clip>
+        </camera>
+      </sensor>
+    </gazebo>
+  </xacro:macro>
+  <xacro:quad_rgb_unit idx="1" y_off="0.030"/>
+  <xacro:quad_rgb_unit idx="2" y_off="0.010"/>
+  <xacro:quad_rgb_unit idx="3" y_off="-0.010"/>
+  <xacro:quad_rgb_unit idx="4" y_off="-0.030"/>
+  <!-- ============================================================ -->
   <!-- Ultrasonic distance sensor (functional)                       -->
   <!-- Modeled after mBot2's real Ultrasonic Sensor 2: output range   -->

Commit message: fix : change position color sensors

File: mbot2_description/urdf/mbot2.urdf.xacro (robot description, xacro)
@@ -32,10 +32,17 @@
   <xacro:property name="us_height" value="0.020"/>
   <xacro:property name="us_mass"   value="0.01"/>
-  <!-- Quad RGB color sensor array, underside of the chassis -->
+  <!-- Front sensor mount plate: extends past the chassis + caster so the -->
+  <!-- Quad RGB array can see the ground ahead of every wheel -->
+  <xacro:property name="mount_length"    value="0.03"/>
+  <xacro:property name="mount_width"     value="0.075"/>
+  <xacro:property name="mount_thickness" value="0.003"/>
+  <xacro:property name="mount_x" value="${chassis_length/2 + mount_length/2}"/>
+  <!-- Quad RGB color sensor array, underside of the front mount plate -->
   <xacro:property name="qrgb_size" value="0.008"/>
   <xacro:property name="qrgb_height" value="0.004"/>
   <xacro:property name="qrgb_mass"   value="0.001"/>
-  <xacro:property name="qrgb_x" value="0.0"/>
+  <xacro:property name="qrgb_x" value="${chassis_length/2 + mount_length - 0.01}"/>
   <xacro:property name="qrgb_z" value="${wheel_radius - qrgb_height/2}"/>
+  <xacro:property name="mount_z" value="${qrgb_z + qrgb_height/2 + mount_thickness/2}"/>
   <!-- Colors -->
   <material name="mbot_blue">
@@ -226,4 +233,26 @@
     <mu2>0.001</mu2>
   </gazebo>
+  <!-- ============================================================ -->
+  <!-- Front sensor mount plate (cosmetic, no collision) — carries   -->
+  <!-- the Quad RGB array out past the caster so the sensors see the -->
+  <!-- ground ahead of every wheel, same as a real line-follower.    -->
+  <!-- ============================================================ -->
+  <link name="sensor_mount_link">
+    <visual>
+      <geometry>
+        <box size="${mount_length} ${mount_width} ${mount_thickness}"/>
+      </geometry>
+      <material name="mbot_dark_grey"/>
+    </visual>
+    <inertial>
+      <mass value="0.002"/>
+      <inertia ixx="1e-8" ixy="0" ixz="0" iyy="1e-8" iyz="0" izz="1e-8"/>
+    </inertial>
+  </link>
+  <joint name="sensor_mount_joint" type="fixed">
+    <parent link="base_link"/>
+    <child link="sensor_mount_link"/>
+    <origin xyz="${mount_x} 0 ${mount_z}" rpy="0 0 0"/>
+  </joint>
   <!-- ============================================================ -->
   <!-- Quad RGB color sensor array (4x), underside of the chassis    -->

Commit message: feat : Make two mBot2s follow each other.

File: mbot2_description/urdf/mbot2.urdf.xacro (robot description, xacro)
@@ -1,4 +1,7 @@
 <?xml version="1.0"?>
 <robot name="mbot2" xmlns:xacro="http://www.ros.org/wiki/xacro">
+  <!-- Prefix ทุก Gazebo topic ของหุ่นแต่ละตัว เช่น /mbot1 หรือ /mbot2 -->
+  <xacro:arg name="robot_namespace" default=""/>
+  <xacro:property name="topic_namespace" value="$(arg robot_namespace)"/>
   <!-- ============================================================ -->
   <!-- Dimensions are approximate, based on mBot2's published        -->
@@ -282,5 +285,5 @@
         <!-- pitch +90deg: rotates the sensor's forward (+x) axis to point straight down (-z) -->
         <pose>0 0 0 0 1.5707963 0</pose>
-        <topic>quad_rgb_${idx}/image</topic>
+        <topic>${topic_namespace}/quad_rgb_${idx}/image</topic>
         <update_rate>15</update_rate>
         <always_on>true</always_on>
@@ -316,5 +319,5 @@
     <sensor name="ultrasonic_sensor" type="gpu_lidar">
       <pose>${us_length/2} 0 0 0 0 0</pose>
-      <topic>ultrasonic/scan</topic>
+      <topic>${topic_namespace}/ultrasonic/scan</topic>
       <update_rate>10</update_rate>
       <always_on>true</always_on>
@@ -348,5 +351,5 @@
   <gazebo reference="cyberpi_link">
     <sensor name="imu_sensor" type="imu">
-      <topic>imu</topic>
+      <topic>${topic_namespace}/imu</topic>
       <update_rate>50</update_rate>
       <always_on>true</always_on>
@@ -365,7 +368,7 @@
       <wheel_radius>${wheel_radius}</wheel_radius>
       <max_linear_acceleration>2.0</max_linear_acceleration>
-      <topic>cmd_vel</topic>
-      <odom_topic>odom</odom_topic>
-      <tf_topic>tf</tf_topic>
+      <topic>${topic_namespace}/cmd_vel</topic>
+      <odom_topic>${topic_namespace}/odom</odom_topic>
+      <tf_topic>${topic_namespace}/tf</tf_topic>
       <frame_id>odom</frame_id>
       <child_frame_id>base_link</child_frame_id>
@@ -374,5 +377,5 @@
     <plugin filename="libignition-gazebo-joint-state-publisher-system.so"
             name="ignition::gazebo::systems::JointStatePublisher">
-      <topic>joint_states</topic>
+      <topic>${topic_namespace}/joint_states</topic>
     </plugin>
   </gazebo>
